Commit message: update model def files for new ref frame and input

File: robot_description_pkg/urdf/robot_0.xacro (robot description, xacro)
@@ -133,5 +133,5 @@
 		<parent link="steering_link_r1"/>
 		<child link="r1_wheel"/>
-		<origin xyz="0 0 ${wheel_radius}" rpy="0 0 0"/>
+		<origin xyz="0 0 ${wheel_radius}" rpy="0 0 -${M_PI_2}"/>
 	</joint>
 	<!-- drive joint r2 -->
@@ -139,5 +139,5 @@
 		<parent link="steering_link_r2"/>
 		<child link="r2_wheel"/>
-		<origin xyz="0 0 ${wheel_radius}" rpy="0 0 0"/>
+		<origin xyz="0 0 ${wheel_radius}" rpy="0 0 -${M_PI_2}"/>
 	</joint>
 	<!-- drive joint l1 -->
@@ -145,5 +145,5 @@
 		<parent link="steering_link_l1"/>
 		<child link="l1_wheel"/>
-		<origin xyz="0 0 ${wheel_radius}" rpy="0 0 0"/>
+		<origin xyz="0 0 ${wheel_radius}" rpy="0 0 -${M_PI_2}"/>
 	</joint>
 	<!-- drive joint l2 -->
@@ -151,5 +151,5 @@
 		<parent link="steering_link_l2"/>
 		<child link="l2_wheel"/>
-		<origin xyz="0 0 ${wheel_radius}" rpy="0 0 0"/>
+		<origin xyz="0 0 ${wheel_radius}" rpy="0 0 -${M_PI_2}"/>
 	</joint>
 	<!-- Transmission: drive, select: effort/vel/pos interfaces -->

Commit message: meerged conflicts

File: robot_description_pkg/urdf/robot_0.xacro (robot description, xacro)
@@ -89,5 +89,5 @@
 		<parent link="left_arm"/>
 		<child link="steering_link_l1"/>
-		<origin xyz="${axis_offset} 0 0" rpy="0 0 0"/>
+		<origin xyz="${axis_offset} 0 0" rpy="0 0 ${M_PI}"/>
 		<axis xyz="0 0 1"/>
 	</joint>
@@ -96,5 +96,5 @@
 		<parent link="left_arm"/>
 		<child link="steering_link_l2"/>
-		<origin xyz="${arm_length-axis_offset} 0 0" rpy="0 0 0"/>
+		<origin xyz="${arm_length-axis_offset} 0 0" rpy="0 0 ${M_PI}"/>
 		<axis xyz="0 0 1"/>
 	</joint>
@@ -103,5 +103,5 @@
 		<parent link="right_arm"/>
 		<child link="steering_link_r1"/>
-		<origin xyz="0 ${axis_offset} 0" rpy="0 0 0"/>
+		<origin xyz="0 ${axis_offset} 0" rpy="0 0 ${M_PI}"/>
 		<axis xyz="0 0 1"/>
 	</joint>
@@ -110,5 +110,5 @@
 		<parent link="right_arm"/>
 		<child link="steering_link_r2"/>
-		<origin xyz="0 ${arm_length-axis_offset} 0" rpy="0 0 0"/>
+		<origin xyz="0 ${arm_length-axis_offset} 0" rpy="0 0 ${M_PI}"/>
 		<axis xyz="0 0 1"/>
 	</joint>

Commit message: updated robot model, inertias and frictions

File: robot_description_pkg/urdf/robot_0.xacro (robot description, xacro)
@@ -5,24 +5,26 @@
 	<xacro:include filename="$(find robot_description_pkg)/urdf/transmission.urdf.xacro" />
 	<xacro:include filename="$(find robot_description_pkg)/urdf/arm.urdf.xacro" />
-	<!-- properties -->
+	<!-- PROPERTIES -->
 	<!--All units in m-kg-s-radians unit system -->
 	<xacro:property name="M_PI" value="3.1415926535897931" />
 	<xacro:property name="M_PI_2" value="1.570796327" />
 	<xacro:property name="DEG_TO_RAD" value="0.017453293" />
-	<!-- friction coefficients -->
-	<xacro:property name="MU_1" value="10000" />
-	<xacro:property name="MU_2" value="10000" />
-	<xacro:property name="arm_mass" value="0.4" />
+	<!-- friction coefficients: https://www.engineeringtoolbox.com/friction-coefficients-d_778.html -->
+	<xacro:property name="MU_1" value="0.8" />
+	<xacro:property name="MU_2" value="0.8" />
+	<!-- mass (kg) -->
+	<xacro:property name="arm_mass" value="10" />
 	<xacro:property name="steer_link_mass" value="0.5" />
-	<xacro:property name="wheel_mass" value="0.3" />
-	<xacro:property name="robot_height" value="0.15" />
+	<xacro:property name="wheel_mass" value="4" />
+	<!-- robot dimensions (m) -->
+	<xacro:property name="robot_height" value="0.2" />
 	<xacro:property name="axis_offset" value="0.125" />
-	<xacro:property name="steer_link_length" value="0.12" />
 	<xacro:property name="steer_link_width" value="0.03" />
-	<xacro:property name="wheel_radius" value="0.05" />
-	<xacro:property name="wheel_width" value="0.03" />
+	<xacro:property name="wheel_radius" value="0.07" />
+	<xacro:property name="wheel_width" value="0.04" />
 	<xacro:property name="arm_length" value="0.6" />
-	<xacro:property name="arm_width" value="0.1" />
-	<xacro:property name="arm_thickness" value="0.025" />
+	<xacro:property name="arm_width" value="0.15" />
+	<xacro:property name="arm_thickness" value="0.1" />
+	<xacro:property name="steer_link_length" value="${arm_thickness/2+wheel_radius}" />
 	 <!-- Macros for calculating inertia -->
 	<xacro:macro name="cylinder_inertia" params="m r h">
