Commit message: added pid gains, breaks gazebo model display and arm locations

File: urdf/robot_0.xacro (robot description, xacro)
@@ -24,7 +24,7 @@
 	<xacro:property name="wheel_width" value="0.04" />
 	<xacro:property name="arm_length" value="0.6" />
+	<xacro:property name="arm_thickness" value="0.1" />
 	<xacro:property name="arm_width" value="0.15" />
-	<xacro:property name="arm_thickness" value="0.1" />
-	<xacro:property name="steer_link_length" value="${arm_thickness/2+wheel_radius}" />
+	<xacro:property name="steer_link_length" value="0.02" /> <!-- ${arm_thickness/2+wheel_radius} -->
 	 <!-- Macros for calculating inertia -->
 	<xacro:macro name="cylinder_inertia" params="m r h">
@@ -56,10 +56,10 @@
 		<turnGravityOff>false</turnGravityOff>
 	</gazebo>
-	<!-- left arm -->
-	<xacro:arm arm_name="left_arm" arm_length="${arm_length}" arm_width="${arm_width}"
+	<!-- x axis arm -->
+	<xacro:arm arm_name="arm_x" arm_length="${arm_length}" arm_width="${arm_width}"
 						arm_thickness="${arm_thickness}" arm_mass="${arm_mass}"
 						rotation_angle="0" X="${(arm_length-arm_width)/2}" Y="0" robot_height="${robot_height}" />
-	<!-- right arm -->
-	<xacro:arm arm_name="right_arm" arm_length="${arm_length}" arm_width="${arm_width}"
+	<!-- y axis arm: shorter to avoid coliision with x axis arm -->
+	<xacro:arm arm_name="arm_y" arm_length="0.5" arm_width="${arm_width}"
 						arm_thickness="${arm_thickness}" arm_mass="${arm_mass}"
 						rotation_angle="${M_PI_2}" X="0" Y="${(arm_length-arm_width)/2}" robot_height="${robot_height}" />
@@ -68,10 +68,10 @@
 		<origin xyz="0 0 0" rpy="0 0 0" />
 		<parent link="base_footprint"/>
-		<child link="left_arm" />
+		<child link="arm_x" />
 	</joint>
 	<joint name="base_footprint_joint_r" type="fixed">
 		<origin xyz="0 0 0" rpy="0 0 0" />
 		<parent link="base_footprint"/>
-		<child link="right_arm" />
+		<child link="arm_y" />
 	</joint>
 	<!-- steering link l1 -->
@@ -89,5 +89,5 @@
 	<!-- yaw joint l1 -->
 	<joint name="yaw_joint_l1" type="continuous">
-		<parent link="left_arm"/>
+		<parent link="arm_x"/>
 		<child link="steering_link_l1"/>
 		<origin xyz="${axis_offset} 0 0" rpy="0 0 ${M_PI}"/>
@@ -96,5 +96,5 @@
 	<!-- yaw joint l2 -->
 	<joint name="yaw_joint_l2" type="continuous">
-		<parent link="left_arm"/>
+		<parent link="arm_x"/>
 		<child link="steering_link_l2"/>
 		<origin xyz="${arm_length-axis_offset} 0 0" rpy="0 0 ${M_PI}"/>
@@ -103,5 +103,5 @@
 	<!-- yaw joint r1 -->
 	<joint name="yaw_joint_r1" type="continuous">
-		<parent link="right_arm"/>
+		<parent link="arm_y"/>
 		<child link="steering_link_r1"/>
 		<origin xyz="0 ${axis_offset} 0" rpy="0 0 ${M_PI}"/>
@@ -110,5 +110,5 @@
 	<!-- yaw joint r2 -->
 	<joint name="yaw_joint_r2" type="continuous">
-		<parent link="right_arm"/>
+		<parent link="arm_y"/>
 		<child link="steering_link_r2"/>
 		<origin xyz="0 ${arm_length-axis_offset} 0" rpy="0 0 ${M_PI}"/>

Commit message: added tofs to sim need to fix publishing the same data. Look slike a gazebo issue

File: urdf/robot_0.xacro (robot description, xacro)
@@ -1,12 +1,19 @@
 <?xml version="1.0"?>
 <robot xmlns:xacro="http://www.ros.org/wiki/xacro" name="AR_0">
+    <!-- robot parts -->
 	<xacro:include filename="$(find ar_sim)/urdf/wheel.urdf.xacro" />
 	<xacro:include filename="$(find ar_sim)/urdf/steering_column.urdf.xacro" />
-	<xacro:include filename="$(find ar_sim)/urdf/transmission.urdf.xacro" />
-	<xacro:include filename="$(find ar_sim)/urdf/arm.urdf.xacro" />
+    <xacro:include filename="$(find ar_sim)/urdf/arm.urdf.xacro" />
+    <!-- actuation -->
+    <xacro:include filename="$(find ar_sim)/urdf/transmission.urdf.xacro" />
+    <!-- sensors -->
+    <xacro:include filename="$(find ar_sim)/urdf/tof.urdf.xacro" />
+    <!-- materials -->
+    <xacro:include filename="$(find ar_sim)/urdf/materials.xacro" />
 	<!-- PROPERTIES -->
 	<!--All units in m-kg-s-radians unit system -->
 	<xacro:property name="M_PI" value="3.1415926535897931" />
-	<xacro:property name="M_PI_2" value="1.570796327" />
+    <xacro:property name="M_PI_2" value="1.570796327" />
+    <xacro:property name="M_PI_4" value="0.7853981635" />
 	<xacro:property name="DEG_TO_RAD" value="0.017453293" />
 	<!-- friction coefficients: https://www.engineeringtoolbox.com/friction-coefficients-d_778.html -->
@@ -26,5 +33,8 @@
 	<xacro:property name="arm_width" value="0.15" />
 	<xacro:property name="arm_thickness" value="0.1" />
-	<xacro:property name="steer_link_length" value="${arm_thickness/2+wheel_radius}" />
+    <xacro:property name="steer_link_length" value="${arm_thickness/2+wheel_radius}" />
+    <!-- sensor properties -->
+    <xacro:property name="TOF_rate" value="30" /> <!-- Hz -->
+    <xacro:property name="visualize_TOFs" value="true" />
 	 <!-- Macros for calculating inertia -->
 	<xacro:macro name="cylinder_inertia" params="m r h">
@@ -36,14 +46,6 @@
 		iyy="${m*(w*w+l*l)/12}" iyz = "0" izz="${m*(h*h+w*w)/12}" />
 	</xacro:macro>
-	<!-- Materials -->
-	<material name="black">
-		<color rgba="0 0 0 1"/>
-	</material>
-	<material name="white">
-		<color rgba="1 1 1 1"/>
-	</material>
-	<!-- BASE-FOOTPRINT -->
- 	<!-- base_footprint is a fictitious link(frame)that is on the ground right below base_link origin -->
-	<link name="base_footprint">
+	<!-- BASE FOOTPRINT -->
+    <link name="base_footprint">
 		<visual>
 			<origin xyz="0 0 0" rpy="0 0 0" />
@@ -178,3 +180,13 @@
 		</plugin>
 	</gazebo>
+    <!-- TOF sensors -->
+    <xacro:tof_sensor name="tof1" parent="tof1_parent_joint" base="base_footprint"
+                      xyz="${arm_thickness} ${arm_thickness} ${robot_height}" rpy="0 0 ${M_PI_4}" rate="${TOF_rate}"
+                      visualize="${visualize_TOFs}"/>
+    <xacro:tof_sensor name="tof2" parent="tof2_parent_joint" base="base_footprint"
+                      xyz="${arm_thickness} ${arm_length-arm_thickness} ${robot_height}" rpy="0 0 0"
+                      rate="${TOF_rate}" visualize="${visualize_TOFs}"/>
+    <xacro:tof_sensor name="tof3" parent="tof3_parent_joint" base="base_footprint"
+                      xyz="${arm_length-arm_thickness} ${arm_thickness} ${robot_height}" rpy="0 0 ${M_PI_2}"
+                      rate="${TOF_rate}" visualize="${visualize_TOFs}"/>
 </robot>

Commit message: tidied up name bug and macro tof fct

File: urdf/robot_0.xacro (robot description, xacro)
@@ -181,12 +181,9 @@
 	</gazebo>
     <!-- TOF sensors -->
-    <xacro:tof_sensor name="tof1" parent="tof1_parent_joint" base="base_footprint"
-                      xyz="${arm_thickness} ${arm_thickness} ${robot_height}" rpy="0 0 ${M_PI_4}" rate="${TOF_rate}"
-                      visualize="${visualize_TOFs}"/>
-    <xacro:tof_sensor name="tof2" parent="tof2_parent_joint" base="base_footprint"
-                      xyz="${arm_thickness} ${arm_length-arm_thickness} ${robot_height}" rpy="0 0 0"
-                      rate="${TOF_rate}" visualize="${visualize_TOFs}"/>
-    <xacro:tof_sensor name="tof3" parent="tof3_parent_joint" base="base_footprint"
-                      xyz="${arm_length-arm_thickness} ${arm_thickness} ${robot_height}" rpy="0 0 ${M_PI_2}"
-                      rate="${TOF_rate}" visualize="${visualize_TOFs}"/>
+    <xacro:tof_sensor name="tof1" base="base_footprint" xyz="${arm_thickness} ${arm_length-arm_thickness} ${robot_height}"
+                      rpy="0 0 0" rate="${TOF_rate}" visualize="${visualize_TOFs}"/>
+    <xacro:tof_sensor name="tof2" base="base_footprint" xyz="${arm_thickness} ${arm_thickness} ${robot_height}"
+                      rpy="0 0 ${M_PI_4}" rate="${TOF_rate}" visualize="${visualize_TOFs}"/>
+    <xacro:tof_sensor name="tof3" base="base_footprint" xyz="${arm_length-arm_thickness} ${arm_thickness} ${robot_height}"
+                      rpy="0 0 ${M_PI_2}" rate="${TOF_rate}" visualize="${visualize_TOFs}"/>
 </robot>

File: urdf/tof.urdf.xacro (robot description, xacro)
@@ -1,7 +1,7 @@
 <?xml version="1.0"?>
 <robot xmlns:xacro="http://www.ros.org/wiki/xacro">
-<xacro:macro name="tof_sensor" params="name parent base xyz rpy rate visualize">
+<xacro:macro name="tof_sensor" params="name base xyz rpy rate visualize">
 <!-- TOF sensor -->
-    <joint name="${parent}" type="fixed">
+    <joint name="${name}_parent_joint" type="fixed">
         <origin xyz="${xyz}" rpy="${rpy}"/>
         <parent link="${base}"/>
@@ -24,5 +24,5 @@
     </link>
     <gazebo reference="${name}">
-        <sensor name="laser" type="ray">
+        <sensor name="${name}" type="ray">
             <pose>0 0 0 0 0 0</pose>
             <ray>
